File: pcbs/corne-v3-cherry/pcb/corne-cherry.kicad_pcb (KiCad board)
At the start: 2 copper layers, 275.5 x 105.6 mm, 172 parts, among them J1 MJ-4PP-9, J2 OLED, J3 MJ-4PP-9, J4 OLED, SW1 SW_PUSH, SW10 SW_PUSH, SW11 SW_PUSH, SW12 SW_PUSH, SW13 SW_PUSH, SW14 SW_PUSH, SW15 SW_PUSH, SW16 SW_PUSH, SW17 SW_PUSH, SW18 SW_PUSH, SW19 SW_PUSH, SW2 SW_PUSH, SW20 SW_PUSH, SW21 SW_PUSH, SW22 SW_PUSH, SW23 SW_PUSH, SW24 SW_PUSH, SW25 SW_PUSH, SW26 SW_PUSH, SW27 SW_PUSH, SW28 SW_PUSH, SW29 SW_PUSH, SW3 SW_PUSH, SW30 SW_PUSH, SW31 SW_PUSH, SW32 SW_PUSH, SW33 SW_PUSH, SW34 SW_PUSH, SW35 SW_PUSH, SW36 SW_PUSH, SW37 SW_PUSH, SW38 SW_PUSH, SW39 SW_PUSH, SW4 SW_PUSH, SW40 SW_PUSH, SW41 SW_PUSH, SW42 SW_PUSH, SW5 SW_PUSH, SW6 SW_PUSH, SW7 SW_PUSH, SW8 SW_PUSH, SW9 SW_PUSH, U1 ProMicro, U2 ProMicro

Commit message: Init 4 key col idea
Parts:
- added D1: D, kbd:D3_SMD_v2, B.Cu at (27.7, 27.7)
- added D22: D, kbd:D3_SMD_v2, B.Cu at (284.2, 17.1)
- added LED34: YS-SK6812MINI-E, kbd:YS-SK6812MINI-E, B.Cu at (276.6, 21.8)
- added LED7: YS-SK6812MINI-E, kbd:YS-SK6812MINI-E, B.Cu at (20.1, 32.4)
- added SW1: SW_PUSH, kbd:CherryMX_Hotswap, F.Cu at (20.1, 27.7)
- added SW22: SW_PUSH, kbd:CherryMX_Hotswap, F.Cu at (276.6, 17.1)
- moved D7 10.9 mm to (27.9, 65.7)
- moved D1 10.9 mm to (27.9, 46.7)
- moved D13 10.9 mm to (27.9, 84.7)
- moved LED13 10.9 mm to (20.2, 70.4)
- moved LED19 10.9 mm to (20.2, 89.4)
- moved LED7 10.9 mm to (20.2, 51.4)
- moved REF** 10.9 mm to (20.3, 94.1)
- moved SW1 10.9 mm to (20.2, 46.7)
- moved SW13 10.9 mm to (20.2, 84.7)
- moved SW7 10.9 mm to (20.2, 65.7)
- moved D22 0.07 mm to (284.3, 35.8)
- moved D28 0.07 mm to (284.3, 54.7)
- moved D34 0.07 mm to (284.3, 73.8)
- moved LED34 0.07 mm to (276.7, 40.6)
- moved LED40 0.07 mm to (276.7, 59.6)
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Routing:
- net row0_r: track 184.4 -> 203.9 mm
- net GND: track 637.2 -> 650.7 mm
- net Net-(LED7-Pad4): track 31.8 -> 42.3 mm, vias 4 -> 6
- net VDD: track 573.1 -> 578.9 mm
- net row0: track 183.2 -> 188.1 mm
- net col1: track 149.4 -> 153.7 mm
- net Net-(D22-Pad2): track 4.05 -> 8.11 mm
- net Net-(D1-Pad2): track 4.04 -> 8.08 mm
- net Net-(LED34-Pad4): track 15.0 -> 18.3 mm
- net Net-(LED13-Pad4): track 33.1 -> 36.1 mm, vias 2 -> 3
- net row2: track 180.7 -> 183.4 mm
- net Net-(LED34-Pad2): track 29.0 -> 31.7 mm, vias 2 -> 3
- net col0_r: track 175.8 -> 178.3 mm, vias 5 -> 6
- net row1: track 193.3 -> 190.9 mm
- net VCC: track 544.3 -> 546.1 mm
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Other:
- board size 275.5 x 105.6 mm -> 275.5 x 109.6 mm
